Commit message: modify the URDF model, start new camera effect

File: install/mecanum_robot/share/mecanum_robot/urdf/mecanum_robot.urdf (robot description, URDF)
Before this commit: robot mecanum_robot, 6 links, 5 joints
Links:
- added link front_left_steering_link, mass 0.1; collision cylinder length=0.05 radius=0.02; visual cylinder length=0.05 radius=0.02
- added link front_right_steering_link, mass 0.1; collision cylinder length=0.05 radius=0.02; visual cylinder length=0.05 radius=0.02
- added link rear_left_steering_link, mass 0.1; collision cylinder length=0.05 radius=0.02; visual cylinder length=0.05 radius=0.02
- added link rear_right_steering_link, mass 0.1; collision cylinder length=0.05 radius=0.02; visual cylinder length=0.05 radius=0.02
- link base_link: mass 5.0 -> 21.0; geometry collision box size=0.508 0.548 0.409; visual box size=0.508 0.548 0.409
- link front_left_wheel: mass 0.3 -> 0.5; geometry collision cylinder length=0.03 radius=0.0625; visual cylinder length=0.03 radius=0.0625
- link front_right_wheel: mass 0.3 -> 0.5; geometry collision cylinder length=0.03 radius=0.0625; visual cylinder length=0.03 radius=0.0625
- link rear_left_wheel: mass 0.3 -> 0.5; geometry collision cylinder length=0.03 radius=0.0625; visual cylinder length=0.03 radius=0.0625
- link rear_right_wheel: mass 0.3 -> 0.5; geometry collision cylinder length=0.03 radius=0.0625; visual cylinder length=0.03 radius=0.0625
Joints:
- added joint front_left_steering_joint: type revolute, parent base_link, child front_left_steering_link, origin xyz=0.1915 0.2115 0.12 rpy=0 0 0, axis 0 0 1, limit lower=-1.5708 upper=1.5708 effort=1000 velocity=10
- added joint front_right_steering_joint: type continuous, parent base_link, child front_right_steering_link, origin xyz=0.1915 -0.2115 0.12 rpy=0 0 0, axis 0 0 1
- added joint rear_left_steering_joint: type continuous, parent base_link, child rear_left_steering_link, origin xyz=-0.1915 0.2115 0.12 rpy=0 0 0, axis 0 0 1
- added joint rear_right_steering_joint: type revolute, parent base_link, child rear_right_steering_link, origin xyz=-0.1915 -0.2115 0.12 rpy=0 0 0, axis 0 0 1, limit lower=-1.5708 upper=1.5708 effort=1000 velocity=10
- joint front_left_wheel_joint: origin xyz=0.2 0.15 0 rpy=0 0 0 -> xyz=0 0 -0.0575 rpy=0 0 0; parent base_link -> front_left_steering_link
- joint front_right_wheel_joint: origin xyz=0.2 -0.15 0 rpy=0 0 0 -> xyz=0 0 -0.0575 rpy=0 0 0; parent base_link -> front_right_steering_link
- joint imu_joint: origin xyz=0 0 0.15 rpy=0 0 0 -> xyz=0 0 0.3245 rpy=0 0 0
- joint rear_left_wheel_joint: origin xyz=-0.2 0.15 0 rpy=0 0 0 -> xyz=0 0 -0.0575 rpy=0 0 0; parent base_link -> rear_left_steering_link
- joint rear_right_wheel_joint: origin xyz=-0.2 -0.15 0 rpy=0 0 0 -> xyz=0 0 -0.0575 rpy=0 0 0; parent base_link -> rear_right_steering_link
